File: Hardware/Eagle/Basic LiPo Charger.brd (EAGLE design)
At the start: 31 x 12.6 mm, 12 parts, among them J1 USB-CON-5PIN-105017-0001, U1 MCP73831

Commit message: Changed resistor value
Parts:
- R1: value 470 -> 120
Changed lines of the file:
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@@
 <?xml version="1.0" encoding="utf-8"?>
 <!DOCTYPE eagle SYSTEM "eagle.dtd">
-<eagle version="8.1.1">
+<eagle version="8.2.0">
 <drawing>
 <settings>
@@
 <attribute name="VALUE" x="31.442" y="52.01" size="0.6096" layer="27" font="vector" ratio="20" rot="R90"/>
 </element>
-<element name="R1" library="NovemberFive-Basic" package="R0603" value="470" x="22.75" y="56.52" smashed="yes" rot="R180"/>
+<element name="R1" library="NovemberFive-Basic" package="R0603" value="120" x="22.75" y="56.52" smashed="yes" rot="R180"/>
 <element name="R2" library="NovemberFive-Basic" package="R0603" value="2K" x="25.4" y="53.34" smashed="yes"/>
 <element name="R3" library="SparkFun-Resistors" package="AXIAL-0.3" value="" x="22.86" y="50.8" smashed="yes">
